File: Motherboard/TinyTendo.kicad_pcb (KiCad board)
At the start: 4 copper layers, 64.7 x 52.2 mm, 47 parts, among them J1 Conn_01x01_Male, J2 Conn_01x01_Male, J3 Conn_01x01_Male, J4 Conn_01x01_Male, J5 Conn_01x01_Male, J6 Conn_01x01_Male, J7 Conn_01x01_Male, J8 Conn_01x01_Male, J9 Conn_01x01_Male, P1 72-Pin Connector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

Commit message: + Motherboard is now V1.0 + Redesigned ScreenReg for improved reliability + Added both versions of ChargeBoost + Remove now redundant files/directories
Other:
- board text added: "Redherring32 2019-2022"
- board text removed: "Redherring32 2021-2022"
Changed lines of the file:
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@@
       (drillshape 0)
       (scaleselection 1)
-      (outputdirectory "K:/Users/Redherring32/Desktop/TinyTendo/Gerbers/Motherboard"))
+      (outputdirectory "../Extract for gerbers/"))
   )
   (net 0 "")
@@
     (effects (font (size 1 1) (thickness 0.15)))
   )
-  (gr_text "Redherring32 2021-2022\n" (at 219.38 123.84) (layer F.SilkS)
+  (gr_text "Redherring32 2019-2022\n" (at 219.38 123.84) (layer F.SilkS)
     (effects (font (size 1 1) (thickness 0.15)))
   )
