File: Supporting PCBs/Button PCB/Button PCB.kicad_pcb (KiCad board)
At the start: 2 copper layers, 82.6 x 41.1 mm, 25 parts, among them U1 CD4021BPW

Commit message: + Motherboard is now V1.0 + Redesigned ScreenReg for improved reliability + Added both versions of ChargeBoost + Remove now redundant files/directories
Routing:
- net /GND: vias 47 -> 46
