File: Supporting PCBs/TNY-NES-Adapter/TNY-NES-Adapter.kicad_pcb (KiCad board)
At the start: 2 copper layers, 2 parts, among them P1 72-Pin Connector, P2 72-Pin Connector

Commit message: + Motherboard is now V1.0 + Redesigned ScreenReg for improved reliability + Added both versions of ChargeBoost + Remove now redundant files/directories
Parts:
- removed the P1 at (180.3, 77.1)
- removed P2: 72-Pin Connector, NESRE:NES_Edge_Connector
- added P1: 72-Pin Connector, NESRE:NES_Edge_Connector, F.Cu at (-33.6, 110.7)
- added P1: 72-Pin Connector, TinyTendo:Cart Slot, F.Cu at (-7.72, 89.7)
Routing:
- net /M2: track 0.00 -> 43.8 mm
- net /CPU-A12: track 0.00 -> 42.0 mm
- net /VCC: track 0.00 -> 40.6 mm
- net /CPU-A13: track 0.00 -> 40.2 mm
- net /CPU-A14: track 0.00 -> 38.4 mm
- net /PPU-D4: track 0.00 -> 38.0 mm
- net /CPU-D7: track 0.00 -> 36.6 mm
- net /PPU-D5: track 0.00 -> 36.2 mm
- net /CPU-D6: track 0.00 -> 34.8 mm
- net /PPU-D6: track 0.00 -> 34.4 mm
- net /CPU-D5: track 0.00 -> 33.0 mm
- net /PPU-D7: track 0.00 -> 32.6 mm
- net /CPU-D4: track 0.00 -> 31.2 mm
- net /PPU-A13: track 0.00 -> 30.8 mm
- net /CPU-D3: track 0.00 -> 29.4 mm
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- added copper zone on B.Cu, net /GND
- added copper zone on F.Cu, net /GND
Other:
- board outline added: 93.4 x 28.2 mm
- board text added: "NES CARTRIDGE LABEL SIDE"
- board text added: "Redhering32 2022"
- board text added: "TNY -> NES Adapter"
