File: Hardware/Button PCB/Button PCB.kicad_pcb (KiCad board)
At the start: 2 copper layers, 82.6 x 41.1 mm, 25 parts, among them U1 CD4021BPW

Commit message: + Corrected duplicate reference error in Chargeboost.sch
+ Made changes to Audio Amp PCB to improve screwpost locations

+ Made changes to Button PCB to improve screwpost locations

+ Moved screen up 6mm to even out bezels on shell

+ Altered shell to improve screwpost placement, and add optional suppport for threaded inserts

+ Added 2 new shell variants, 1 with a logo via multicolor printing and threaded inserts, 1 with just threaded inserts
Parts:
- moved   8.50 mm to (83.9, -40.6)
- moved Red 3.78 mm to (79.8, -53.7)
- moved White 3.78 mm to (79.8, -62.1)
- moved Brown 3.78 mm to (79.7, -45.2)
- moved Orange 3.78 mm to (79.8, -49.4)
- moved Yellow 3.78 mm to (79.8, -57.9)
- moved   3.00 mm to (67.2, -61.8)
- moved   3.00 mm to (5.24, -63.4)
Routing:
- net /Clock: track 36.6 -> 42.2 mm
- net /Strobe: track 35.4 -> 37.8 mm
- net /Data: track 59.5 -> 61.8 mm
- net /GND: track 0.00 -> 0.78 mm
Other:
- board size 82.6 x 41.1 mm -> 82.6 x 44.1 mm
- net class Default removed
